File: pcb/IR.kicad_sch (KiCad schematic)
At the start: 6 parts, among them Q10 BS170, Q11 TEFT4300

Commit message: Did fan wiring
Parts:
- R21: value 40 -> 36
Connections:
- net +3.3V: no longer D6.A
- new net +5V: D6.A
Changed lines of the file:
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@@
 	(wire
 		(pts
-			(xy 86.36 49.53) (xy 86.36 48.26)
+			(xy 86.36 46.99) (xy 86.36 49.53)
 		)
 		(stroke
@@
 			)
 		)
-		(property "Value" "40"
+		(property "Value" "36"
 			(at 88.9 68.5799 0)
 			(show_name no)
@@
 	)
 	(symbol
-		(lib_id "power:+3.3V")
-		(at 86.36 48.26 0)
-		(unit 1)
-		(body_style 1)
-		(exclude_from_sim no)
-		(in_bom yes)
-		(on_board yes)
-		(in_pos_files yes)
-		(dnp no)
-		(fields_autoplaced yes)
-		(property "Reference" "#PWR052"
-			(at 86.36 52.07 0)
-			(hide yes)
-			(show_name no)
-			(do_not_autoplace no)
-			(effects
-				(font
-					(size 1.27 1.27)
-				)
-			)
-		)
-		(property "Value" "+3.3V"
-			(at 86.36 43.18 0)
-			(show_name no)
-			(do_not_autoplace no)
-			(effects
-				(font
-					(size 1.27 1.27)
-				)
-			)
-		)
-		(property "Footprint" ""
-			(at 86.36 48.26 0)
-			(hide yes)
-			(show_name no)
-			(do_not_autoplace no)
-			(effects
-				(font
-					(size 1.27 1.27)
-				)
-			)
-		)
-		(property "Datasheet" ""
-			(at 86.36 48.26 0)
-			(hide yes)
-			(show_name no)
-			(do_not_autoplace no)
-			(effects
-				(font
-					(size 1.27 1.27)
-				)
-			)
-		)
-		(property "Description" "Power symbol creates a global label with name \"+3.3V\""
-			(at 86.36 48.26 0)
-			(hide yes)
-			(show_name no)
-			(do_not_autoplace no)
-			(effects
-				(font
-					(size 1.27 1.27)
-				)
-			)
-		)
-		(pin "1"
-		)
-		(instances
-			(project "micromouse-pcb"
-				(path "/6bab3514-b9e6-4652-bd2e-edc57bdbde3d/1ceefd87-148b-487c-9cc8-0976f70f8c92"
-					(reference "#PWR055")
-					(unit 1)
-				)
-				(path "/6bab3514-b9e6-4652-bd2e-edc57bdbde3d/5dec74b7-7e95-4967-a373-cc0339326363"
-					(reference "#PWR063")
-					(unit 1)
-				)
-				(path "/6bab3514-b9e6-4652-bd2e-edc57bdbde3d/7f4b8bd4-4b33-4dde-a793-226b8e2de73f"
-					(reference "#PWR052")
-					(unit 1)
-				)
-				(path "/6bab3514-b9e6-4652-bd2e-edc57bdbde3d/9892aae5-d20a-4a72-957e-b0df2200cbe7"
-					(reference "#PWR059")
-					(unit 1)
-				)
-			)
-		)
-	)
-	(symbol
 		(lib_id "power:GND")
 		(at 86.36 86.36 0)
@@
 					(unit 1)
 				)
+			)
+		)
+	)
+	(symbol
+		(lib_id "power:+5V")
+		(at 86.36 46.99 0)
+		(unit 1)
+		(body_style 1)
+		(exclude_from_sim no)
+		(in_bom yes)
+		(on_board yes)
+		(in_pos_files yes)
+		(dnp no)
+		(fields_autoplaced yes)
+		(property "Reference" "#PWR02"
+			(at 86.36 50.8 0)
+			(hide yes)
+			(show_name no)
+			(do_not_autoplace no)
+			(effects
+				(font
+					(size 1.27 1.27)
+				)
+			)
+		)
+		(property "Value" "+5V"
+			(at 86.36 41.91 0)
+			(show_name no)
+			(do_not_autoplace no)
+			(effects
+				(font
+					(size 1.27 1.27)
+				)
+			)
+		)
+		(property "Footprint" ""
+			(at 86.36 46.99 0)
+			(hide yes)
+			(show_name no)
+			(do_not_autoplace no)
+			(effects
+				(font
+					(size 1.27 1.27)
+				)
+			)
+		)
+		(property "Datasheet" ""
+			(at 86.36 46.99 0)
+			(hide yes)
+			(show_name no)
+			(do_not_autoplace no)
+			(effects
+				(font
+					(size 1.27 1.27)
+				)
+			)
+		)
+		(property "Description" "Power symbol creates a global label with name \"+5V\""
+			(at 86.36 46.99 0)
+			(hide yes)
+			(show_name no)
+			(do_not_autoplace no)
+			(effects
+				(font
+					(size 1.27 1.27)
+				)
+			)
+		)
+		(pin "1"
+		)
+		(instances
+			(project "micromouse-pcb"
+				(path "/6bab3514-b9e6-4652-bd2e-edc57bdbde3d/1ceefd87-148b-487c-9cc8-0976f70f8c92"
+					(reference "#PWR06")
+					(unit 1)
+				)
+				(path "/6bab3514-b9e6-4652-bd2e-edc57bdbde3d/5dec74b7-7e95-4967-a373-cc0339326363"
+					(reference "#PWR09")
+					(unit 1)
+				)
+				(path "/6bab3514-b9e6-4652-bd2e-edc57bdbde3d/7f4b8bd4-4b33-4dde-a793-226b8e2de73f"
+					(reference "#PWR02")
+					(unit 1)
+				)
+				(path "/6bab3514-b9e6-4652-bd2e-edc57bdbde3d/9892aae5-d20a-4a72-957e-b0df2200cbe7"
+					(reference "#PWR07")
+					(unit 1)
+				)
